Commit message: Add link_prefix argument to robot's xacro
Because parameter tf_prefix doesn't be supported in ROS Noetic anymore.
I tried some repo fix this problem, but the tf_prefix has problem on planar_move_plugins.
So the simple way is add prefix on xacro.

File: gazebo/robot_description/urdf/simple-omni-robot.xacro (robot description, xacro)
@@ -1,4 +1,6 @@
 <?xml version="1.0" encoding="utf-8"?>
 <robot xmlns:xacro="http://www.ros.org/wiki/xacro" name="simple_omni_robot">
+  <!-- robot_state_publisher no longer support tf_prefix in ROS Noetic...-->
+  <xacro:arg name="link_prefix" default="" />
   <xacro:include filename="$(find hector_sensors_description)/urdf/hokuyo_utm30lx.urdf.xacro" />
   <xacro:include filename="$(find robot_description)/urdf/simple-omni-robot.gazebo" />
@@ -6,5 +8,5 @@
   <xacro:property name="RADIUS" value="0.105" />
   <xacro:property name="HEIGHT" value="0.192" />
-  <xacro:hokuyo_utm30lx name="lidar" parent="base_link" ros_topic="laser"
+  <xacro:hokuyo_utm30lx name="$(arg link_prefix)/lidar" parent="$(arg link_prefix)/base_link" ros_topic="laser"
                         update_rate="30" ray_count="270"
                         min_angle="-135" max_angle="135">
@@ -13,5 +15,5 @@
   </xacro:hokuyo_utm30lx>
   <!-- Links -->
-  <link name="head">
+  <link name="$(arg link_prefix)/head">
     <visual>
       <origin xyz="0 0 0" rpy="0 0 0" />
@@ -21,5 +23,5 @@
     </visual>
   </link>
-  <link name="base_footprint">
+  <link name="$(arg link_prefix)/base_footprint">
     <visual>
       <origin xyz="0 0 0" rpy="0 0 0" />
@@ -29,5 +31,5 @@
     </visual>
   </link>
-  <link name="base_link">
+  <link name="$(arg link_prefix)/base_link">
     <inertial>
       <!-- <origin xyz="0 0 ${HEIGHT/2}" rpy="0 0 0" /> -->
@@ -72,12 +74,12 @@
   <joint name="head_joint" type="fixed">
     <origin xyz="${RADIUS} 0 ${HEIGHT/2}" rpy="0 0 0" />
-    <parent link="base_link"/>
-    <child link="head" />
+    <parent link="$(arg link_prefix)/base_link"/>
+    <child link="$(arg link_prefix)/head" />
   </joint>
   <joint name="base_link_joint" type="fixed">
     <origin xyz="0.0 0 ${HEIGHT/2}" rpy="0 0 0" />
-    <parent link="base_footprint"/>
-    <child link="base_link" />
+    <parent link="$(arg link_prefix)/base_footprint"/>
+    <child link="$(arg link_prefix)/base_link" />
   </joint>
-  <xacro:simple_omni_robot_gazebo />
+  <xacro:simple_omni_robot_gazebo prefix="$(arg link_prefix)" />
 </robot>

Commit message: Modified robot's model, let it float on the ground little bit.

File: gazebo/robot_description/urdf/simple-omni-robot.xacro (robot description, xacro)
@@ -25,5 +25,5 @@
   <link name="$(arg link_prefix)/base_footprint">
     <visual>
-      <origin xyz="0 0 0" rpy="0 0 0" />
+      <origin xyz="0 0 0.005" rpy="0 0 0" />
       <geometry>
         <cylinder radius="${RADIUS}" length="0.01" />
@@ -64,8 +64,8 @@
       </geometry>
     </visual>
-    <collision name="collision">
+    <collision name="baselink">
       <origin xyz="0 0 0" rpy="0 0 0" />
       <geometry>
-        <cylinder radius="${RADIUS}" length="${HEIGHT}" />
+        <cylinder radius="${RADIUS}" length="${HEIGHT+0.05}" />
       </geometry>
     </collision>
@@ -78,5 +78,5 @@
   </joint>
   <joint name="base_link_joint" type="fixed">
-    <origin xyz="0.0 0 ${HEIGHT/2}" rpy="0 0 0" />
+    <origin xyz="0.0 0 ${HEIGHT/2+0.01}" rpy="0 0 0" />
     <parent link="$(arg link_prefix)/base_footprint"/>
     <child link="$(arg link_prefix)/base_link" />

Commit message: Colorful robots
use 'gazebo_ros_model_color' with distinct colors 'colors.yaml'

File: gazebo/robot_description/urdf/simple-omni-robot.xacro (robot description, xacro)
@@ -3,4 +3,5 @@
   <!-- robot_state_publisher no longer support tf_prefix in ROS Noetic...-->
   <xacro:arg name="link_prefix" default="" />
+  <xacro:arg name="id_num" default="" />
   <xacro:include filename="$(find hector_sensors_description)/urdf/hokuyo_utm30lx.urdf.xacro" />
   <xacro:include filename="$(find robot_description)/urdf/simple-omni-robot.gazebo" />
@@ -11,6 +12,6 @@
                         update_rate="30" ray_count="270"
                         min_angle="-135" max_angle="135">
-    <!-- Place lidar on the top and back of robot, lidar size is W60xD60xH87mm -->
-    <origin xyz="${RADIUS*-1+0.03} 0.0 ${HEIGHT/2+0.0435}" rpy="0 0 0" />
+  <!-- Place lidar on the top and back of robot, lidar size is W60xD60xH87mm -->
+  <origin xyz="${RADIUS*-1+0.03} 0.0 ${HEIGHT/2+0.0435}" rpy="0 0 0" />
   </xacro:hokuyo_utm30lx>
   <!-- Links -->
@@ -82,4 +83,4 @@
     <child link="$(arg link_prefix)/base_link" />
   </joint>
-  <xacro:simple_omni_robot_gazebo prefix="$(arg link_prefix)" />
+  <xacro:simple_omni_robot_gazebo prefix="$(arg link_prefix)" id_num="$(arg id_num)" />
 </robot>
